File: mcu.kicad_sch (KiCad schematic)
At the start: 8 parts, among them J2 SWD, J3 ESP-01S, U4 STM32F411RETx, Y1 10MHz

Commit message: ESP module pins
Changed lines of the file:
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@@
+	)
+	(label "ESP_RST"
+		(at 129.54 63.5 0)
+		(effects
+			(font
+				(size 1.27 1.27)
+			)
+			(justify left bottom)
+		)
 	)
 	(label "ESP_RST"
 		(at 195.58 29.21 90)
+		(effects
+			(font
+				(size 1.27 1.27)
+			)
+			(justify left bottom)
+		)
+	)
+	(label "ESP_RX"
+		(at 129.54 55.88 0)
 		(effects
 			(font
@@
 	)
 	(label "ESP_PD"
+		(at 129.54 60.96 0)
+		(effects
+			(font
+				(size 1.27 1.27)
+			)
+			(justify left bottom)
+		)
+	)
+	(label "ESP_PD"
 		(at 193.04 29.21 90)
 		(effects
@@
 		(effects
 			(font
+				(size 1.27 1.27)
+			)
+			(justify left bottom)
+		)
+	)
+	(label "ESP_TX"
+		(at 129.54 58.42 0)
+		(effects
+			(font

Commit message: update
- fixed what the switching mixer sees when the input is "disabled" - tied to 1/2*3.3V instead of GND
- added another J-FET transistor to the AGC loop
Parts:
- renumbered C12 to C13, C11 to C14, J2 to J1, J3 to J2, R8 to R11, R7 to R12
Other:
- company: (none) -> Wojciech Kaczmarski SP5WWP
Changed lines of the file:
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@@
 	(title_block
 		(title "PCSK225 time signal receiver")
-		(date "2026-09-05")
+		(date "2026-10-24")
+		(company "Wojciech Kaczmarski SP5WWP")
 	)
 	(text "Confirm orientation!"
@@
 		(in_pos_files yes)
 		(dnp no)
-		(property "Reference" "R7"
+		(property "Reference" "R12"
 			(at 71.12 58.42 90)
 			(show_name no)
@@
 			(project "pcsk225_ntp"
 				(path "/ece5592d-c78f-4d56-a72a-26347184f54b/3d2e24f8-47c2-47c7-92ad-c9b6c073ed55"
-					(reference "R7")
+					(reference "R12")
 					(unit 1)
 				)
@@
 		(dnp no)
 		(fields_autoplaced yes)
-		(property "Reference" "C12"
+		(property "Reference" "C13"
 			(at 26.67 44.4499 0)
 			(show_name no)
@@
 			(project "pcsk225_ntp"
 				(path "/ece5592d-c78f-4d56-a72a-26347184f54b/3d2e24f8-47c2-47c7-92ad-c9b6c073ed55"
-					(reference "C12")
+					(reference "C13")
 					(unit 1)
 				)
@@
 		(dnp no)
 		(fields_autoplaced yes)
-		(property "Reference" "#PWR025"
+		(property "Reference" "#PWR027"
 			(at 35.56 77.47 0)
 			(hide yes)
@@
 			(project "pcsk225_ntp"
 				(path "/ece5592d-c78f-4d56-a72a-26347184f54b/3d2e24f8-47c2-47c7-92ad-c9b6c073ed55"
-					(reference "#PWR025")
+					(reference "#PWR027")
 					(unit 1)
 				)
@@
 		(dnp no)
 		(fields_autoplaced yes)
-		(property "Reference" "#PWR024"
+		(property "Reference" "#PWR032"
 			(at 99.06 143.51 0)
 			(hide yes)
@@
 			(project "pcsk225_ntp"
 				(path "/ece5592d-c78f-4d56-a72a-26347184f54b/3d2e24f8-47c2-47c7-92ad-c9b6c073ed55"
-					(reference "#PWR024")
+					(reference "#PWR032")
 					(unit 1)
 				)
@@
 		(dnp no)
 		(fields_autoplaced yes)
-		(property "Reference" "#PWR030"
+		(property "Reference" "#PWR033"
 			(at 190.5 50.8 0)
 			(hide yes)
@@
 			(project "pcsk225_ntp"
 				(path "/ece5592d-c78f-4d56-a72a-26347184f54b/3d2e24f8-47c2-47c7-92ad-c9b6c073ed55"
-					(reference "#PWR030")
+					(reference "#PWR033")
 					(unit 1)
 				)
@@
 		(dnp no)
 		(fields_autoplaced yes)
-		(property "Reference" "#PWR029"
+		(property "Reference" "#PWR023"
 			(at 22.86 44.45 0)
 			(hide yes)
@@
 			(project "pcsk225_ntp"
 				(path "/ece5592d-c78f-4d56-a72a-26347184f54b/3d2e24f8-47c2-47c7-92ad-c9b6c073ed55"
-					(reference "#PWR029")
+					(reference "#PWR023")
 					(unit 1)
 				)
@@
 		(dnp no)
 		(fields_autoplaced yes)
-		(property "Reference" "#PWR020"
+		(property "Reference" "#PWR030"
 			(at 66.04 60.96 0)
 			(hide yes)
@@
 			(project "pcsk225_ntp"
 				(path "/ece5592d-c78f-4d56-a72a-26347184f54b/3d2e24f8-47c2-47c7-92ad-c9b6c073ed55"
-					(reference "#PWR020")
+					(reference "#PWR030")
 					(unit 1)
 				)
@@
 		(dnp no)
 		(fields_autoplaced yes)
-		(property "Reference" "#PWR028"
+		(property "Reference" "#PWR024"
 			(at 22.86 57.15 0)
 			(hide yes)
@@
 			(project "pcsk225_ntp"
 				(path "/ece5592d-c78f-4d56-a72a-26347184f54b/3d2e24f8-47c2-47c7-92ad-c9b6c073ed55"
-					(reference "#PWR028")
+					(reference "#PWR024")
 					(unit 1)
 				)
@@
 		(dnp no)
 		(fields_autoplaced yes)
-		(property "Reference" "#PWR023"
+		(property "Reference" "#PWR031"
 			(at 96.52 41.91 0)
 			(hide yes)
@@
 			(project "pcsk225_ntp"
 				(path "/ece5592d-c78f-4d56-a72a-26347184f54b/3d2e24f8-47c2-47c7-92ad-c9b6c073ed55"
-					(reference "#PWR023")
+					(reference "#PWR031")
 					(unit 1)
 				)
@@
 		(dnp no)
 		(fields_autoplaced yes)
-		(property "Reference" "C11"
+		(property "Reference" "C14"
 			(at 48.26 55.88 90)
 			(show_name no)
@@
 			(project "pcsk225_ntp"
 				(path "/ece5592d-c78f-4d56-a72a-26347184f54b/3d2e24f8-47c2-47c7-92ad-c9b6c073ed55"
-					(reference "C11")
+					(reference "C14")
 					(unit 1)
 				)
@@
 		(in_pos_files yes)
 		(dnp no)
-		(property "Reference" "R8"
+		(property "Reference" "R11"
 			(at 71.12 43.18 90)
 			(show_name no)
@@
 			(project "pcsk225_ntp"
 				(path "/ece5592d-c78f-4d56-a72a-26347184f54b/3d2e24f8-47c2-47c7-92ad-c9b6c073ed55"
-					(reference "R8")
+					(reference "R11")
 					(unit 1)
 				)
@@
 		(dnp no)
 		(fields_autoplaced yes)
-		(property "Reference" "J3"
+		(property "Reference" "J2"
 			(at 200.66 35.5599 90)
 			(show_name no)
@@
 			(project "pcsk225_ntp"
 				(path "/ece5592d-c78f-4d56-a72a-26347184f54b/3d2e24f8-47c2-47c7-92ad-c9b6c073ed55"
-					(reference "J3")
+					(reference "J2")
 					(unit 1)
 				)
@@
 		(dnp no)
 		(fields_autoplaced yes)
-		(property "Reference" "J2"
+		(property "Reference" "J1"
 			(at 43.18 17.78 0)
 			(show_name no)
@@
 			(project "pcsk225_ntp"
 				(path "/ece5592d-c78f-4d56-a72a-26347184f54b/3d2e24f8-47c2-47c7-92ad-c9b6c073ed55"
-					(reference "J2")
+					(reference "J1")
 					(unit 1)
 				)
@@
 		(dnp no)
 		(fields_autoplaced yes)
-		(property "Reference" "#PWR021"
+		(property "Reference" "#PWR029"
 			(at 66.04 50.8 0)
 			(hide yes)
@@
 			(project "pcsk225_ntp"
 				(path "/ece5592d-c78f-4d56-a72a-26347184f54b/3d2e24f8-47c2-47c7-92ad-c9b6c073ed55"
-					(reference "#PWR021")
+					(reference "#PWR029")
 					(unit 1)
 				)
@@
 		(dnp no)
 		(fields_autoplaced yes)
-		(property "Reference" "#PWR031"
+		(property "Reference" "#PWR034"
 			(at 198.12 33.02 0)
 			(hide yes)
@@
 			(project "pcsk225_ntp"
 				(path "/ece5592d-c78f-4d56-a72a-26347184f54b/3d2e24f8-47c2-47c7-92ad-c9b6c073ed55"
-					(reference "#PWR031")
+					(reference "#PWR034")
 					(unit 1)
 				)
@@
 		(dnp no)
 		(fields_autoplaced yes)
-		(property "Reference" "#PWR022"
+		(property "Reference" "#PWR028"
 			(at 49.53 39.37 0)
 			(hide yes)
@@
 			(project "pcsk225_ntp"
 				(path "/ece5592d-c78f-4d56-a72a-26347184f54b/3d2e24f8-47c2-47c7-92ad-c9b6c073ed55"
-					(reference "#PWR022")
+					(reference "#PWR028")
 					(unit 1)
 				)
@@
 		(dnp no)
 		(fields_autoplaced yes)
-		(property "Reference" "#PWR027"
+		(property "Reference" "#PWR025"
 			(at 26.67 71.12 0)
 			(hide yes)
@@
 			(project "pcsk225_ntp"
 				(path "/ece5592d-c78f-4d56-a72a-26347184f54b/3d2e24f8-47c2-47c7-92ad-c9b6c073ed55"
-					(reference "#PWR027")
+					(reference "#PWR025")
 					(unit 1)
 				)
