File: pcsk225_ntp.kicad_sch (KiCad schematic)
At the start: 0 parts

Commit message: update
- fixed what the switching mixer sees when the input is "disabled" - tied to 1/2*3.3V instead of GND
- added another J-FET transistor to the AGC loop
Other:
- company: (none) -> Wojciech Kaczmarski SP5WWP
Changed lines of the file:
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@@
 	(title_block
 		(title "PCSK225 time signal receiver")
-		(date "2026-09-05")
-		(comment 1 "Drawn by Wojciech SP5WWP")
+		(date "2026-10-24")
+		(company "Wojciech Kaczmarski SP5WWP")
 	)
 	(wire
